Commit message: added 2d viz, modified urdf model, need to implement contour following

File: models/block_big.urdf (robot description, URDF)
Before this commit: robot block_2, 1 links, 0 joints
Links:
- link block_2_base_link: geometry collision box size=0.15 0.15 0.05; visual box size=0.15 0.15 0.05

Commit message: rough probing code done. need to follow contour

File: models/block_big.urdf (robot description, URDF)
Before this commit: robot block_2, 1 links, 0 joints
Links:
- link block_2_base_link: mass 0.02 -> 2.0

Commit message: basic contour following, error after two sides

File: models/block_big.urdf (robot description, URDF)
Before this commit: robot block_2, 1 links, 0 joints
Links:
- link block_2_base_link: geometry collision box size=0.10 0.10 0.05; visual box size=0.10 0.10 0.05
