Commit message: concave object collision doesn't work for non-static objects :(

File: models/shapes/hex.urdf (robot description, URDF)
Before this commit: robot butter, 1 links, 0 joints
Links:
- removed link butter_base_link
- added link hex_base_link, mass 0.9827; collision mesh filename=hex.stl scale=1.0 1.0 2.0; visual mesh filename=hex.stl scale=1.0 1.0 2.0
