Commit message: updated physical parameters, need to get plotting for all objects

File: models/shapes/tri1.urdf (robot description, URDF)
Before this commit: robot rect1, 1 links, 0 joints
Links:
- removed link rect1_base_link
- added link tri1_base_link, mass 0.8028; collision mesh filename=tri1.stl scale=1.0 1.0 2.0; visual mesh filename=tri1.stl scale=1.0 1.0 2.0

File: models/shapes/tri2.urdf (robot description, URDF)
Before this commit: robot rect1, 1 links, 0 joints
Links:
- removed link rect1_base_link
- added link tri2_base_link, mass 0.9826; collision mesh filename=tri2.stl scale=1.0 1.0 2.0; visual mesh filename=tri2.stl scale=1.0 1.0 2.0

File: models/shapes/tri3.urdf (robot description, URDF)
Before this commit: robot rect1, 1 links, 0 joints
Links:
- removed link rect1_base_link
- added link tri3_base_link, mass 1.1326; collision mesh filename=tri3.stl scale=1.0 1.0 2.0; visual mesh filename=tri3.stl scale=1.0 1.0 2.0
