Commit message: debugging forces

File: models/shapes/ellip1.urdf (robot description, URDF)
Before this commit: robot ellip1, 1 links, 0 joints
Links:
- link ellip1_base_link: geometry collision mesh filename=ellip1.stl scale=1.0 1.0 1.0; visual mesh filename=ellip1.stl scale=1.0 1.0 1.0

File: models/shapes/pusher.urdf (robot description, URDF)
Before this commit: robot rect1, 1 links, 0 joints
Links:
- removed link rect1_base_link
- added link pusher_base_link, mass 0.8; collision mesh filename=ellip1.stl scale=0.1 0.1 1.0; visual mesh filename=ellip1.stl scale=0.1 0.1 1.0
