Commit message: further debugging

File: models/shapes/pusher.urdf (robot description, URDF)
Before this commit: robot pusher, 1 links, 0 joints
Links:
- link pusher_base_link: geometry collision cylinder length=0.01275 radius=0.010; visual cylinder length=0.01275 radius=0.010

Commit message: trying two prongs

File: models/shapes/pusher.urdf (robot description, URDF)
Before this commit: robot pusher, 1 links, 0 joints
Links:
- removed link pusher_base_link
- added link pusher_1, mass 0.8; collision cylinder length=0.01275 radius=0.005; visual cylinder length=0.01275 radius=0.005
- added link pusher_2, mass 0.8; collision cylinder length=0.01275 radius=0.005; visual cylinder length=0.01275 radius=0.005
- added link pusher_base, mass 0.8
Joints:
- added joint pusher_1_joint: type fixed, parent pusher_base, child pusher_1, origin xyz=0.02 0 0 rpy=0 0 0, axis 0 0 1
- added joint pusher_2_joint: type fixed, parent pusher_base, child pusher_2, origin xyz=-0.02 0 0 rpy=0 0 0, axis 0 0 1

Commit message: changed radius and dimensions, contact threshold, force_plotter works for two prongs

File: models/shapes/pusher.urdf (robot description, URDF)
Before this commit: robot pusher, 3 links, 2 joints
Links:
- link pusher_1: mass 0.8 -> 0.5; geometry collision cylinder length=0.015 radius=0.00313; visual cylinder length=0.015 radius=0.00313
- link pusher_2: mass 0.8 -> 0.5; geometry collision cylinder length=0.015 radius=0.00313; visual cylinder length=0.015 radius=0.00313
Joints:
- joint pusher_1_joint: origin xyz=0.02 0 0 rpy=0 0 0 -> xyz=0.02 0 -0.0075 rpy=0 0 0
- joint pusher_2_joint: origin xyz=-0.02 0 0 rpy=0 0 0 -> xyz=-0.02 0 -0.0075 rpy=0 0 0
