Commit message: added other models and modified sim

File: models/kuka_iiwa/model.urdf (robot description, URDF)
Before this commit: robot lbr_iiwa, 9 links, 8 joints
Links:
- link iiwa_link_ee: geometry collision cylinder length=0.1275 radius=0.010; visual cylinder length=0.1275 radius=0.010

File: models/shapes/ellip3.urdf (robot description, URDF)
Before this commit: robot rect, 1 links, 0 joints
Links:
- removed link rect_base_link
- added link ellip3_base_link, mass 1.3338; collision mesh filename=ellip3.stl scale=1.0 1.0 2.0; visual mesh filename=ellip3.stl scale=1.0 1.0 2.0

File: models/shapes/rect1.urdf (robot description, URDF)
Before this commit: robot rect, 1 links, 0 joints
Links:
- removed link rect_base_link
- added link rect1_base_link, mass 0.8374; collision mesh filename=rect1.stl scale=1.0 1.0 2.0; visual mesh filename=rect1.stl scale=1.0 1.0 2.0

File: models/shapes/rect2.urdf (robot description, URDF)
Before this commit: robot ellip, 1 links, 0 joints
Links:
- removed link ellip_base_link
- added link rect2_base_link, mass 1.045; collision mesh filename=rect2.stl scale=1.0 1.0 2.0; visual mesh filename=rect2.stl scale=1.0 1.0 2.0

Commit message: modified urdfs, using simple_sim.py for now

File: models/kuka_iiwa/model.urdf (robot description, URDF)
Before this commit: robot lbr_iiwa, 9 links, 8 joints
Links:
- link iiwa_link_ee: mass None -> 0.8

File: models/shapes/butter.urdf (robot description, URDF)
Before this commit: robot butter, 1 links, 0 joints
Links:
- link butter_base_link: geometry collision mesh filename=butter.stl scale=1.0 1.0 1.0; visual mesh filename=butter.stl scale=1.0 1.0 1.0

File: models/shapes/ellip2.urdf (robot description, URDF)
Before this commit: robot ellip2, 1 links, 0 joints
Links:
- link ellip2_base_link: geometry collision mesh filename=ellip2.stl scale=1.0 1.0 1.0; visual mesh filename=ellip2.stl scale=1.0 1.0 1.0

File: models/shapes/ellip3.urdf (robot description, URDF)
Before this commit: robot ellip3, 1 links, 0 joints
Links:
- link ellip3_base_link: geometry collision mesh filename=ellip3.stl scale=1.0 1.0 1.0; visual mesh filename=ellip3.stl scale=1.0 1.0 1.0

File: models/shapes/hex.urdf (robot description, URDF)
Before this commit: robot hex, 1 links, 0 joints
Links:
- link hex_base_link: geometry collision mesh filename=hex.stl scale=1.0 1.0 1.0; visual mesh filename=hex.stl scale=1.0 1.0 1.0

File: models/shapes/rect1.urdf (robot description, URDF)
Before this commit: robot rect1, 1 links, 0 joints
Links:
- link rect1_base_link: geometry collision mesh filename=rect1.stl scale=1.0 1.0 1.0; visual mesh filename=rect1.stl scale=1.0 1.0 1.0

File: models/shapes/rect2.urdf (robot description, URDF)
Before this commit: robot rect2, 1 links, 0 joints
Links:
- link rect2_base_link: geometry collision mesh filename=rect2.stl scale=1.0 1.0 1.0; visual mesh filename=rect2.stl scale=1.0 1.0 1.0

File: models/shapes/rect3.urdf (robot description, URDF)
Before this commit: robot rect3, 1 links, 0 joints
Links:
- link rect3_base_link: geometry collision mesh filename=rect3.stl scale=1.0 1.0 1.0; visual mesh filename=rect3.stl scale=1.0 1.0 1.0

File: models/shapes/tri1.urdf (robot description, URDF)
Before this commit: robot tri1, 1 links, 0 joints
Links:
- link tri1_base_link: geometry collision mesh filename=tri1.stl scale=1.0 1.0 1.0; visual mesh filename=tri1.stl scale=1.0 1.0 1.0

File: models/shapes/tri2.urdf (robot description, URDF)
Before this commit: robot tri2, 1 links, 0 joints
Links:
- link tri2_base_link: geometry collision mesh filename=tri2.stl scale=1.0 1.0 1.0; visual mesh filename=tri2.stl scale=1.0 1.0 1.0

File: models/shapes/tri3.urdf (robot description, URDF)
Before this commit: robot tri3, 1 links, 0 joints
Links:
- link tri3_base_link: geometry collision mesh filename=tri3.stl scale=1.0 1.0 1.0; visual mesh filename=tri3.stl scale=1.0 1.0 1.0
